File: pcb/avr-co2-detector.kicad_sch (KiCad schematic)
At the start: 63 parts, among them J1 USB TYPE-C, J2 Backlight, J3 Backlight, J4 LCD0802, J5 AVR-ISP-10, J6 "Debug UART", J7 "ESP-Prog", SW1 "Reset AVR", SW2 "Reset ESP", SW3 "Config"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

Commit message: Added GND TestPoint, assigned revision 2, updated Gerber and drill files
Parts:
- added TP1: GND TestPoint, TestPoint:TestPoint_Bridge_Pitch2.54mm_Drill1.0mm, symbol Connector:TestPoint
Connections:
- net GND: now also TP1.1
Changed lines of the file:
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@@
   (junction (at 135.89 31.75) (diameter 0) (color 0 0 0 0)
   )
+  (junction (at 143.51 88.9) (diameter 0) (color 0 0 0 0)
+  )
   (junction (at 165.1 128.27) (diameter 0) (color 0 0 0 0)
   )
@@
     (stroke (width 0) (type default) (color 0 0 0 0))
   )
-  (wire (pts (xy 171.45 88.9) (xy 138.43 88.9))
-    (stroke (width 0) (type default) (color 0 0 0 0))
-  )
   (wire (pts (xy 58.42 133.35) (xy 69.85 133.35))
     (stroke (width 0) (type default) (color 0 0 0 0))
@@
     (stroke (width 0) (type default) (color 0 0 0 0))
   )
+  (wire (pts (xy 143.51 88.9) (xy 138.43 88.9))
+    (stroke (width 0) (type default) (color 0 0 0 0))
+  )
   (wire (pts (xy 250.19 101.6) (xy 267.97 101.6))
     (stroke (width 0) (type default) (color 0 0 0 0))
@@
     (stroke (width 0) (type default) (color 0 0 0 0))
   )
+  (wire (pts (xy 143.51 88.9) (xy 171.45 88.9))
+    (stroke (width 0) (type default) (color 0 0 0 0))
+  )
   (wire (pts (xy 351.79 156.21) (xy 351.79 180.34))
     (stroke (width 0) (type default) (color 0 0 0 0))
@@
     (pin "1")
   )
+  (symbol (lib_id "Connector:TestPoint") (at 143.51 88.9 180) (unit 1)
+    (in_bom yes) (on_board yes) (fields_autoplaced)
+    (property "Reference" "TP1" (id 0) (at 146.05 90.9319 0)
+      (effects (font (size 1.27 1.27)) (justify right))
+    )
+    (property "Value" "GND TestPoint" (id 1) (at 146.05 93.4719 0)
+      (effects (font (size 1.27 1.27)) (justify right))
+    )
+    (property "Footprint" "TestPoint:TestPoint_Bridge_Pitch2.54mm_Drill1.0mm" (id 2) (at 138.43 88.9 0)
+      (effects (font (size 1.27 1.27)) hide)
+    )
+    (property "Datasheet" "~" (id 3) (at 138.43 88.9 0)
+      (effects (font (size 1.27 1.27)) hide)
+    )
+    (pin "1")
+  )
   (symbol (lib_id "Device:C_Polarized_Small") (at 189.23 49.53 0) (unit 1)
     (in_bom yes) (on_board yes) (fields_autoplaced)
@@
       (reference "SW3") (unit 1) (value "\"Config\"") (footprint "Button_Switch_SMD:SW_Push_1P1T_NO_6x6mm_H9.5mm")
     )
+    (path "/32cd2556-3e5e-4e66-84bc-4d4104f89375"
+      (reference "TP1") (unit 1) (value "GND TestPoint") (footprint "TestPoint:TestPoint_Bridge_Pitch2.54mm_Drill1.0mm")
+    )
     (path "/4b3936fe-90f3-4535-9194-6fd9522a5a05"
